File: interface-swd.kicad_sch (KiCad schematic)
At the start: 1 part, among them J5 Conn_02x05_Odd_Even

Commit message: Creating fab package
Parts:
- J5: value Conn_02x05_Odd_Even -> Conn_02x05_Odd_Even Male; Supplier_1 Price @ Qty (none) -> 0.33515; Supplier_1 Unit Price 0.54 -> 0.95000
Changed lines of the file:
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@@
 			)
 		)
-		(property "Value" "Conn_02x05_Odd_Even"
+		(property "Value" "Conn_02x05_Odd_Even Male"
 			(at 149.86 87.63 0)
 			(effects
@@
 			)
 		)
-		(property "Supplier_1 Unit Price" "0.54"
+		(property "Supplier_1 Unit Price" "0.95000"
 			(at 148.59 96.52 0)
 			(effects
@@
 			)
 		)
-		(property "Supplier_1 Price @ Qty" ""
+		(property "Supplier_1 Price @ Qty" "0.33515"
 			(at 148.59 96.52 0)
 			(effects
