File: interface-usd.kicad_sch (KiCad schematic)
At the start: 1 part, among them J8 MEM2075-00-140-01-A

Commit message: Fixing footprint imports
Parts:
- J8: footprint MEM2075-00-140-01-A:GCT_MEM2075-00-140-01-A -> footprints:GCT_MEM2075-00-140-01-A
Changed lines of the file:
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@@
 			)
 		)
-		(property "Footprint" "MEM2075-00-140-01-A:GCT_MEM2075-00-140-01-A"
+		(property "Footprint" "footprints:GCT_MEM2075-00-140-01-A"
 			(at 142.24 88.9 0)
 			(effects

Commit message: Spamming 0 ohm resistors
Parts:
- added R23: 0, Resistor_SMD:R_0603_1608Metric, symbol Device:R
Connections:
- net +3V3: now also R23.1; no longer J8.P4 (VDD)
- new net: J8.P4 (VDD), R23.2
Changed lines of the file:
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@@
+	(wire
+		(pts
+			(xy 173.99 81.28) (xy 177.8 81.28)
+		)
+		(stroke
+			(width 0)
+			(type default)
+		)
+	)
 	(wire
 		(pts
@@
 	(wire
 		(pts
-			(xy 160.02 81.28) (xy 177.8 81.28)
+			(xy 160.02 81.28) (xy 166.37 81.28)
 		)
 		(stroke
@@
 	(wire
 		(pts
-			(xy 160.02 88.9) (xy 167.64 88.9)
+			(xy 160.02 88.9) (xy 179.07 88.9)
 		)
 		(stroke
@@
 	)
 	(label "SPI.MOSI"
-		(at 106.68 83.82 0)
+		(at 111.76 83.82 0)
 		(fields_autoplaced yes)
 		(effects
@@
 	)
 	(label "SPI.SCK"
-		(at 106.68 81.28 0)
+		(at 111.76 81.28 0)
 		(fields_autoplaced yes)
 		(effects
@@
 	)
 	(label "SPI.MISO"
-		(at 106.68 86.36 0)
+		(at 111.76 86.36 0)
 		(fields_autoplaced yes)
 		(effects
@@
 	(hierarchical_label "CARD_DETECT"
 		(shape output)
-		(at 167.64 88.9 0)
+		(at 179.07 88.9 0)
 		(fields_autoplaced yes)
 		(effects
@@
 		)
 	)
+	(symbol
+		(lib_id "Device:R")
+		(at 170.18 81.28 270)
+		(unit 1)
+		(exclude_from_sim no)
+		(in_bom yes)
+		(on_board yes)
+		(dnp no)
+		(property "Reference" "R23"
+			(at 166.37 79.756 90)
+			(effects
+				(font
+					(size 1.27 1.27)
+				)
+			)
+		)
+		(property "Value" "0"
+			(at 170.18 81.28 90)
+			(effects
+				(font
+					(size 1.27 1.27)
+					(thickness 0.254)
+					(bold yes)
+				)
+			)
+		)
+		(property "Footprint" "Resistor_SMD:R_0603_1608Metric"
+			(at 170.18 79.502 90)
+			(effects
+				(font
+					(size 1.27 1.27)
+				)
+				(hide yes)
+			)
+		)
+		(property "Datasheet" "Datasheet"
+			(at 170.18 81.28 0)
+			(effects
+				(font
+					(size 1.27 1.27)
+				)
+				(hide yes)
+			)
+		)
+		(property "Description" "Resistor"
+			(at 170.18 81.28 0)
+			(effects
+				(font
+					(size 1.27 1.27)
+				)
+				(hide yes)
+			)
+		)
+		(property "Mfr" "YAGEO"
+			(at 170.18 81.28 0)
+			(effects
+				(font
+					(size 1.27 1.27)
+				)
+				(hide yes)
+			)
+		)
+		(property "Mfr P/N" "RC0603JR-070RL"
+			(at 170.18 81.28 0)
+			(effects
+				(font
+					(size 1.27 1.27)
+				)
+				(hide yes)
+			)
+		)
+		(property "Supplier_1" "Digikey"
+			(at 170.18 81.28 0)
+			(effects
+				(font
+					(size 1.27 1.27)
+				)
+				(hide yes)
+			)
+		)
+		(property "Supplier_1 P/N" "311-0.0GRCT-ND"
+			(at 170.18 81.28 0)
+			(effects
+				(font
+					(size 1.27 1.27)
+				)
+				(hide yes)
+			)
+		)
+		(property "Supplier_1 Unit Price" "$0.10000 "
+			(at 170.18 81.28 0)
+			(effects
+				(font
+					(size 1.27 1.27)
+				)
+				(hide yes)
+			)
+		)
+		(property "Supplier_1 Price @ Qty" "$0.00304 "
+			(at 170.18 81.28 0)
+			(effects
+				(font
+					(size 1.27 1.27)
+				)
+				(hide yes)
+			)
+		)
+		(property "Supplier_2" ""
+			(at 170.18 81.28 0)
+			(effects
+				(font
+					(size 1.27 1.27)
+				)
+				(hide yes)
+			)
+		)
+		(property "Supplier_2 P/N" ""
+			(at 170.18 81.28 0)
+			(effects
+				(font
+					(size 1.27 1.27)
+				)
+				(hide yes)
+			)
+		)
+		(property "Supplier_2 Unit Price" ""
+			(at 170.18 81.28 0)
+			(effects
+				(font
+					(size 1.27 1.27)
+				)
+				(hide yes)
+			)
+		)
+		(property "Supplier_2 Price @ Qty" ""
+			(at 170.18 81.28 0)
+			(effects
+				(font
+					(size 1.27 1.27)
+				)
+				(hide yes)
+			)
+		)
+		(pin "1"
+		)
+		(pin "2"
+		)
+		(instances
+			(project "roamer"
+				(path "/1c59de6a-87fe-4223-8898-4b0383164a31/544d54f1-dde3-4fcc-ac29-865cf5bd110b"
+					(reference "R23")
+					(unit 1)
+				)
+			)
+		)
+	)

Commit message: Adding more 0 ohm resistors and pullups for I2C lines
Parts:
- added R34: 10K, Resistor_SMD:R_0603_1608Metric, symbol Device:R
- R23: value 0 -> 10K; Mfr YAGEO -> Stackpole Electronics Inc; Mfr P/N RC0603JR-070RL -> RNCP0603FTD10K0; Supplier_1 P/N 311-0.0GRCT-ND -> RNCP0603FTD10K0CT-ND; Supplier_1 Price @ Qty $0.00304 -> 0.0170; Supplier_1 Unit Price $0.10000 -> 0.10
Connections:
- net +3V3: now also J8.P4 (VDD), R34.1; no longer R23.1
- net CARD_DETECT: now also R34.2
- net CS_uSD: now also R23.2
- net GND: now also R23.1

Commit message: Adding diodes for Air Quality Sensor SET and RESET pins
Connections:
- net CARD_DETECT renamed uSD_DETECT
Changed lines of the file:
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@@
 		)
 	)
-	(hierarchical_label "CARD_DETECT"
+	(hierarchical_label "uSD_DETECT"
 		(shape output)
 		(at 179.07 88.9 0)

Commit message: Starting layout
Connections:
- net uSD_DETECT: no longer names the net of J8.P9 (CD), R34.2
- no-connect marks 2 -> 3
Other:
- note added: "Can place a uSD_DETECT label here"
Changed lines of the file:
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@@
 		(at 121.92 91.44)
+	)
+	(no_connect
+		(at 179.07 88.9)
 	)
 	(bus_entry
@@
 			(width 0)
 			(type default)
+		)
+	)
+	(text "Can place a uSD_DETECT label here"
+		(exclude_from_sim no)
+		(at 198.882 89.154 0)
+		(effects
+			(font
+				(size 1.27 1.27)
+			)
 		)
 	)
@@
 		)
 	)
-	(hierarchical_label "uSD_DETECT"
-		(shape output)
-		(at 179.07 88.9 0)
-		(fields_autoplaced yes)
-		(effects
-			(font
-				(size 1.27 1.27)
-			)
-			(justify left)
-		)
-	)

Commit message: Creating fab package
Parts:
- J8: Supplier_1 Unit Price $2.44 -> 2.44
Changed lines of the file:
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@@
 			)
 		)
-		(property "Supplier_1 Unit Price" "$2.44"
+		(property "Supplier_1 Unit Price" "2.44"
 			(at 142.24 88.9 0)
 			(effects
