File: sensor-current.kicad_sch (KiCad schematic)
At the start: 9 parts, among them U8 INA260

Commit message: Adding finishing touches
Parts:
- removed TP8, TP9: TestPoint, TestPoint:TestPoint_Loop_D2.50mm_Drill1.0mm, symbol Connector:TestPoint

Commit message: Creating fab package
Parts:
- R16, R17, R18, R19, R21: Supplier_1 Price @ Qty $0.00304 -> 0.00304; Supplier_1 Unit Price $0.10000 -> 0.10000
- U8: Supplier_1 Price @ Qty $2.85475 -> 2.77257; Supplier_1 Unit Price $5.43000 -> 4.86000
Changed lines of the file:
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@@
 			)
 		)
-		(property "Supplier_1 Unit Price" "$0.10000 "
+		(property "Supplier_1 Unit Price" "0.10000 "
 			(at 127 95.25 0)
 			(effects
@@
 			)
 		)
-		(property "Supplier_1 Price @ Qty" "$0.00304 "
+		(property "Supplier_1 Price @ Qty" "0.00304 "
 			(at 127 95.25 0)
 			(effects
@@
 			)
 		)
-		(property "Supplier_1 Unit Price" "$0.10000 "
-			(at 173.99 97.79 0)
-			(effects
-				(font
-					(size 1.27 1.27)
-				)
-				(hide yes)
-			)
-		)
-		(property "Supplier_1 Price @ Qty" "$0.00304 "
+		(property "Supplier_1 Unit Price" "0.10000 "
+			(at 173.99 97.79 0)
+			(effects
+				(font
+					(size 1.27 1.27)
+				)
+				(hide yes)
+			)
+		)
+		(property "Supplier_1 Price @ Qty" "0.00304 "
 			(at 173.99 97.79 0)
 			(effects
@@
 			)
 		)
-		(property "Supplier_1 Unit Price" "$5.43000"
-			(at 151.13 100.33 0)
-			(effects
-				(font
-					(size 1.27 1.27)
-				)
-				(hide yes)
-			)
-		)
-		(property "Supplier_1 Price @ Qty" "$2.85475"
+		(property "Supplier_1 Unit Price" "4.86000"
+			(at 151.13 100.33 0)
+			(effects
+				(font
+					(size 1.27 1.27)
+				)
+				(hide yes)
+			)
+		)
+		(property "Supplier_1 Price @ Qty" "2.77257"
 			(at 151.13 100.33 0)
 			(effects
@@
 			)
 		)
-		(property "Supplier_1 Unit Price" "$0.10000 "
-			(at 127 105.41 0)
-			(effects
-				(font
-					(size 1.27 1.27)
-				)
-				(hide yes)
-			)
-		)
-		(property "Supplier_1 Price @ Qty" "$0.00304 "
+		(property "Supplier_1 Unit Price" "0.10000 "
+			(at 127 105.41 0)
+			(effects
+				(font
+					(size 1.27 1.27)
+				)
+				(hide yes)
+			)
+		)
+		(property "Supplier_1 Price @ Qty" "0.00304 "
 			(at 127 105.41 0)
 			(effects
@@
 			)
 		)
-		(property "Supplier_1 Unit Price" "$0.10000 "
-			(at 151.13 73.66 0)
-			(effects
-				(font
-					(size 1.27 1.27)
-				)
-				(hide yes)
-			)
-		)
-		(property "Supplier_1 Price @ Qty" "$0.00304 "
+		(property "Supplier_1 Unit Price" "0.10000 "
+			(at 151.13 73.66 0)
+			(effects
+				(font
+					(size 1.27 1.27)
+				)
+				(hide yes)
+			)
+		)
+		(property "Supplier_1 Price @ Qty" "0.00304 "
 			(at 151.13 73.66 0)
 			(effects
@@
 			)
 		)
-		(property "Supplier_1 Unit Price" "$0.10000 "
+		(property "Supplier_1 Unit Price" "0.10000 "
 			(at 173.99 100.33 0)
 			(effects
@@
 			)
 		)
-		(property "Supplier_1 Price @ Qty" "$0.00304 "
+		(property "Supplier_1 Price @ Qty" "0.00304 "
 			(at 173.99 100.33 0)
 			(effects
